File: PHYS/PHYS 4050H/Kicad Schematics/MeasurementSwitching.kicad_sch (KiCad schematic)
At the start: 18 parts, among them U4 Sine Generator IC, U5 L7805, U6 SN74HC4066N, U7 TL081, Y2 16.0MHz

Commit message: .
Parts:
- removed C12: 0.1u, symbol Device:C
- removed C8, C9: 10u, symbol Device:C_Polarized
- removed D2: LED_PWR, symbol Device:LED
- removed R5: 220, symbol Device:R
- removed U5: L7805, symbol Regulator_Linear:L7805
- U4: value Sine Generator IC -> Switching IC
Connections:
- net 5V: now reaches R4.2, U4.20 (AVCC), U4.21 (AREF), U4.7 (VCC), U6.14 (VCC)
Other:
- note removed: "TODO: LPF Here for AVCC?"
