File: PHYS/PHYS 4050H/Kicad Schematics/Kicad Schematics.kicad_sch (KiCad schematic)
At the start: 15 parts, among them U1 Sine Generator IC, U2 MCP4822, U3 L7805, Y1 16.0MHz

Commit message: .
Parts:
- removed C2: 10u (tantalum), symbol Device:C_Polarized
- added U8: ${SIM.PARAMS}, symbol Simulation_SPICE:OPAMP
Connections:
- net SINE: now also U8.1 (+), U8.5
- net V+: now also U8.3 (V+)
- net 5V: now reaches C1.1, C5.1, R2.2, R3.2, U1.20 (AVCC), U1.7 (VCC), U2.1 (Vdd), U3.3 (OUT)
- net 5V: no longer U1.21 (AREF)
- new net V-: U8.4 (V-)
Other:
- note removed: "TODO: LPF Here for AVCC?"
- moved on the sheet: C4, C5, D1, R2, U3

Commit message: more
Connections:
- net SINE: now also U8.2 (-); no longer C3.1, R1.2, U8.1 (+)
- new net: C3.1, R1.2, U8.1 (+)
Changed lines of the file:
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@@
+	)
+	(junction
+		(at 219.71 41.91)
+		(diameter 0)
+		(color 0 0 0 0)
 	)
 	(junction
@@
 	)
 	(junction
-		(at 218.44 41.91)
-		(diameter 0)
-		(color 0 0 0 0)
-	)
-	(junction
 		(at 52.07 157.48)
 		(diameter 0)
@@
 	)
 	(junction
-		(at 195.58 39.37)
-		(diameter 0)
-		(color 0 0 0 0)
-	)
-	(junction
 		(at 91.44 68.58)
 		(diameter 0)
@@
 	(wire
 		(pts
+			(xy 219.71 57.15) (xy 219.71 41.91)
+		)
+		(stroke
+			(width 0)
+			(type default)
+		)
+	)
+	(wire
+		(pts
 			(xy 49.53 182.88) (xy 52.07 182.88)
 		)
@@
 	(wire
 		(pts
-			(xy 195.58 39.37) (xy 203.2 39.37)
-		)
-		(stroke
-			(width 0)
-			(type default)
-		)
-	)
-	(wire
-		(pts
-			(xy 195.58 39.37) (xy 195.58 25.4)
-		)
-		(stroke
-			(width 0)
-			(type default)
-		)
-	)
-	(wire
-		(pts
 			(xy 31.75 157.48) (xy 31.75 165.1)
 		)
@@
 	(wire
 		(pts
+			(xy 219.71 41.91) (xy 229.87 41.91)
+		)
+		(stroke
+			(width 0)
+			(type default)
+		)
+	)
+	(wire
+		(pts
 			(xy 52.07 182.88) (xy 71.12 182.88)
 		)
@@
 	(wire
 		(pts
-			(xy 218.44 25.4) (xy 218.44 41.91)
-		)
-		(stroke
-			(width 0)
-			(type default)
-		)
-	)
-	(wire
-		(pts
 			(xy 185.42 54.61) (xy 185.42 46.99)
 		)
@@
 	(wire
 		(pts
+			(xy 200.66 44.45) (xy 200.66 57.15)
+		)
+		(stroke
+			(width 0)
+			(type default)
+		)
+	)
+	(wire
+		(pts
 			(xy 64.77 68.58) (xy 66.04 68.58)
 		)
@@
 	(wire
 		(pts
-			(xy 185.42 39.37) (xy 195.58 39.37)
-		)
-		(stroke
-			(width 0)
-			(type default)
-		)
-	)
-	(wire
-		(pts
-			(xy 218.44 41.91) (xy 229.87 41.91)
+			(xy 185.42 39.37) (xy 203.2 39.37)
+		)
+		(stroke
+			(width 0)
+			(type default)
+		)
+	)
+	(wire
+		(pts
+			(xy 218.44 41.91) (xy 219.71 41.91)
 		)
 		(stroke
@@
 	(wire
 		(pts
-			(xy 195.58 25.4) (xy 218.44 25.4)
-		)
-		(stroke
-			(width 0)
-			(type default)
-		)
-	)
-	(wire
-		(pts
 			(xy 73.66 68.58) (xy 91.44 68.58)
 		)
@@
 	(wire
 		(pts
+			(xy 203.2 44.45) (xy 200.66 44.45)
+		)
+		(stroke
+			(width 0)
+			(type default)
+		)
+	)
+	(wire
+		(pts
 			(xy 52.07 157.48) (xy 52.07 165.1)
 		)
@@
 		(pts
 			(xy 80.01 43.18) (xy 85.09 43.18)
+		)
+		(stroke
+			(width 0)
+			(type default)
+		)
+	)
+	(wire
+		(pts
+			(xy 200.66 57.15) (xy 219.71 57.15)
 		)
 		(stroke
@@
 		(on_board yes)
 		(dnp no)
-		(fields_autoplaced yes)
 		(property "Reference" "U8"
-			(at 218.44 36.7598 0)
-			(effects
-				(font
+			(at 213.36 45.974 0)
+			(effects
+				(font
